File: VehicleCurrentSense_PCB/VehicleCurrentSense_PCB.kicad_pcb (KiCad board)
At the start: 4 copper layers, 90 x 35 mm, 65 parts, among them J1 Conn_01x07, J2 USB_B, J3 Test Current, Q1 BC847BS, U1 HAIS 100-P, U10 LMV321, U11 TL331, U2 MCP3426-xSN, U3 AMS1117-3.3, U5 USBLC6-2SC6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

Commit message: Submitted for Manufacturing
Other:
- board text added: "JLCJLCJLCJLC"

Commit message: Optimised
Parts:
- removed D6: Green, LED_SMD:LED_0603_1608Metric
- removed J2: USB_B, Connector_USB:USB_Micro-B_Molex-105017-0001
- removed R15, R16: 4.7k, Resistor_SMD:R_0603_1608Metric
- removed R29: 4.2k, Resistor_SMD:R_0603_1608Metric
- added C8: 100n, Capacitor_SMD:C_0603_1608Metric, F.Cu at (137.0, 94.7)
- added D1: 771-PLVA650A, Package_TO_SOT_SMD:SOT-23, F.Cu at (187.9, 72.0)
- added J4: USB_B_Micro, Connector_USB:USB_Micro-B_Wuerth_614105150721_Vertical, F.Cu at (172.8, 102.7)
- added R2: 3.3k, Resistor_SMD:R_0603_1608Metric, F.Cu at (141.3, 92.3)
- C4: value 100n -> 1u
- R17, R18, R19, R20: moved to F.Cu
- U2: value MCP3426-xSN -> LMV321; footprint Package_SO:SOIC-8_3.9x4.9mm_P1.27mm -> Package_TO_SOT_SMD:SOT-23-5
- moved U2 19.4 mm to (137.4, 92.2), turned to 180 degrees
- moved C4 15.2 mm to (141.3, 93.8), turned to 0 degrees
- moved R19 12.9 mm to (145.2, 93.8), turned to 0 degrees
- moved R17 11.4 mm to (145.2, 90.8), turned to 0 degrees
- moved R20 11.0 mm to (145.2, 95.3), turned to 180 degrees
- moved R18 9.35 mm to (145.2, 92.3), turned to 180 degrees
- moved C16 5.70 mm to (141.3, 85.7)
- moved C17 5.70 mm to (145.2, 87.8)
- moved C18 5.70 mm to (145.2, 84.8)
- moved C20 5.70 mm to (141.3, 82.7)
- moved C5 5.70 mm to (137.7, 80.8)
- moved C6 5.70 mm to (141.3, 84.2)
- moved R1 5.70 mm to (136.2, 80.8)
- moved R22 5.70 mm to (137.1, 89.7)
- moved R23 5.70 mm to (137.1, 86.7)
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Connections:
- C4 pad 1: +5V -> Net-(U2-+)
- J1 pad 2: Local -> Upstream
- J1 pad 3: Upstream -> Local
- R19 pad 1: VREF -> VREF_OUT
- R22 pad 2: VREF -> VREF_OUT
- U2 pad 1: LEM_OUT -> Net-(U2-+)
- U2 pad 3: +5V -> VREF_OUT
- U2 pad 4: SDA -> VREF_OUT
- U2 pad 5: SCL -> +5V
- U5 pad 4: D- Out -> D-
- U5 pad 6: D+ Out -> D+
- U7 pad 23: SCL -> unconnected-(U7-IO15-Pad23)
- U7 pad 24: unconnected-(U7-IO2-Pad24) -> 3V3 LEM_OUT
- U7 pad 26: SDA -> 3V3 VREF
- U7 pad 31: 3V3 VREF -> unconnected-(U7-IO19-Pad31)
- U7 pad 33: 3V3 LEM_OUT -> unconnected-(U7-IO21-Pad33)
- U7 pad 6: Local -> Upstream
- U7 pad 7: Upstream -> Local
- U8 pad 5: D+ Out -> D+
- U8 pad 6: D- Out -> D-
Routing:
- net VREF: track 74.8 -> 23.4 mm, vias 1 -> 2
- net LEM_OUT: track 51.4 -> 22.9 mm
- net D-: track 2.69 -> 19.1 mm, vias 0 -> 2
- net VREF_OUT: track 0.00 -> 13.5 mm, vias 0 -> 2
- net SCL: track 11.4 -> 0.00 mm
- net D+: track 5.26 -> 16.4 mm
- net 3V3 LEM_OUT: track 10.0 -> 18.3 mm, vias 1 -> 0
- net SDA: track 7.28 -> 0.00 mm
- net D+ Out: track 6.78 -> 0.00 mm
- net D- Out: track 6.51 -> 0.00 mm
- net BSPD Threshold: track 28.4 -> 34.1 mm, vias 0 -> 1
- net Net-(U2-+): track 0.00 -> 4.00 mm
- net Net-(U1-OUTPUT): track 12.2 -> 15.9 mm
- net BSPD: track 57.1 -> 53.6 mm
- net 3V3 VREF: track 13.0 -> 16.2 mm, vias 1 -> 0
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Other:
- board text added: "locked"
- board text removed: ">5kW"
- board text removed: "TEST CURRENT"
