File: VehicleCurrentSense_PCB/VehicleCurrentSense_PCB.kicad_sch (KiCad schematic)
At the start: 65 parts, among them J1 Conn_01x07, J1 USB_B, J3 Test Current, Q1 BC847BS, U1 AMS1117-3.3, U1 HAIS 100-P, U11 TL331, U13 LMV321, U2 MCP3426-xSN, U5 CH340C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

Commit message: Optimised
Parts:
- removed D5: Green, LED_SMD:LED_0603_1608Metric, symbol Device:LED_Small
- removed J1: USB_B, Connector_USB:USB_Micro-B_Molex-105017-0001, symbol Connector:USB_B
- removed R31: 4.2k, Resistor_SMD:R_0603_1608Metric, symbol Device:R_Small
- removed R8 (x2): 4.7k, Resistor_SMD:R_0603_1608Metric, symbol Device:R_Small
- removed U2: MCP3426-xSN, Package_SO:SOIC-8_3.9x4.9mm_P1.27mm, symbol Analog_ADC:MCP3426-xSN
- added C8: 100n, Capacitor_SMD:C_0603_1608Metric, symbol Device:C_Small
- added D3: 771-PLVA650A, Package_TO_SOT_SMD:SOT-23, symbol Device:D_Zener
- added J4: USB_B_Micro, Connector_USB:USB_Micro-B_Wuerth_614105150721_Vertical, symbol Connector:USB_B_Micro
- added R2: 3.3k, Resistor_SMD:R_0603_1608Metric, symbol Device:R_Small
- added U2: LMV321, Package_TO_SOT_SMD:SOT-23-5, symbol Amplifier_Operational:LMV321
- C4: value 100n -> 1u
Connections:
- net D+ Out is gone; now on net D+: U5.5 (UD+), U7.6 (I/O1)
- net D- Out is gone; now on net D-: U5.6 (UD-), U7.4 (I/O2)
- net SDA is gone; now on net 3V3 VREF: U6.26 (IO4)
- net +5V: now also C8.1, U2.5 (V+); no longer C4.1
- net 3V3 LEM_OUT: now also U6.24 (IO2); no longer U6.33 (IO21)
- net 3V3 VREF: no longer U6.31 (IO19)
- net D+: now also J4.3 (D+)
- net D-: now also J4.2 (D-)
- net GND: now also C8.2, D3.1 (A), J4.5 (GND), U2.2 (V-)
- net Local: now also J1.3 (Pin_3), U6.7 (IO35); no longer J1.2 (Pin_2), U6.6 (IO34)
- net Upstream: now also J1.2 (Pin_2), U6.6 (IO34); no longer J1.3 (Pin_3), U6.7 (IO35)
- net VREF: now also R2.1; no longer R22.2, R8.1
- net at D1.2 (A): now also J4.1 (VBUS)
- net at C1.1, C1.1, F1.2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: now also D3.3 (K)
- net SCL: no longer names the net of U6.23 (IO15)
- new net: C4.1, R2.2, U2.1 (+)
- new net VREF_OUT: R22.2, R8.1, U2.3 (-), U2.4
- no-connect marks 27 -> 30
Other:
- moved on the sheet: C1, C2, C3, C5, C6, D1, F1, J1, J3, R1, TP3, U1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
