File: VehicleJunctionBoxMotherboard_PCB/VehicleJunctionBoxMotherboard_PCB.kicad_pcb (KiCad board)
At the start: 4 copper layers, 100 x 100 mm, 121 parts, among them J1 HVD IL, J2 Vehicle, J3 TSMP+, J4 TSMP-, J5 HV+, J6 HV-, J7 TSMP GLV-, J9 Conn_01x07, Q1 IXTY1R6N100D2, Q3 FDMS86255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

Commit message: Submitted for Manufacturing
Other:
- board text added: "+5V"
- board text added: "1"
- board text added: "12"
- board text added: "1: GLV+ 2: BSPD Test + 3: BSPD Test - 4: GND 5: DOC Fault 6: TSAL Green 7: TSAL Red 8: BSPD 9: CAN+ 10: CAN- 11: SD Loop In 12: SD Loop Out"
- board text added: "6"
- board text added: "7"
- board text added: "9"
- board text added: "9: BSPD Test - 8: BSPD Test + 7: GND 6: BSPD 5: CAN+ 4: CAN- 3: Upstream 2: Local 1: +5V"
- board text added: ">60V"
- board text added: "CURRENT SENSOR"
- board text added: "DISCHARGE"
- board text added: "DISCHARGE THRESHOLD"
- board text added: "DOC"
- board text added: "GND"
- board text added: "GRN"
- board text added: "HV"
- board text added: "HV+"
- board text added: "HV-"
- board text added: "HVD INTERLOCK"
- board text added: "JLCJLCJLCJLC"
- board text added: "Junction Box Motherboard TSAL, DISCHARGE, PDOC"
- board text added: "LV"
- board text added: "Niko Smith"
- board text added: "RED"
- board text added: "THRESHOLD"
- board text added: "TSAL"
- board text added: "TSMP+"
- board text added: "TSMP-"
- board text removed: "locked"

Commit message: Optimised
Parts:
- removed C29, C30: 100n, Capacitor_SMD:C_0603_1608Metric
- removed R34, R38: 5.6k, Resistor_SMD:R_0603_1608Metric
- removed R36, R40, R45, R46: 10k, Resistor_SMD:R_0603_1608Metric
- removed REF** (x2): Symbol_HighVoltage_Type2_CopperTop_VerySmall, Symbol:Symbol_HighVoltage_Type2_CopperTop_VerySmall
- removed U11, U14: TLV7031DBV, Package_TO_SOT_SMD:SOT-23-5
- added D11: 771-PLVA650A, Package_TO_SOT_SMD:SOT-23, F.Cu at (54.4, 102.6)
- added D12: Green, LED_SMD:LED_0603_1608Metric, F.Cu at (92.1, 94.5)
- R41, R42: value 10k -> 18k
- R5: value 10k -> 4.7k
- moved R43 7.35 mm to (39.7, 77.3)
- moved R41 4.45 mm to (39.7, 78.8)
- moved R39 3.05 mm to (39.7, 75.8)
- moved R42 3.05 mm to (39.7, 74.4)
Connections:
- J9 pad 2: Local -> Upstream
- J9 pad 3: Upstream -> Local
- R39 pad 1: Net-(U11-+) -> Upstream
- R41 pad 2: Net-(U14-+) -> Local
- R42 pad 2: Net-(U11-+) -> Upstream
- R43 pad 1: Net-(U14-+) -> Local
- R5 pad 2: GLV+ -> Net-(D12-K)
Routing:
- net Thresh: track 21.0 -> 0.00 mm
- net +5V: track 37.3 -> 31.5 mm, vias 18 -> 15
- net GLV+: track 68.4 -> 72.3 mm
- net Net-(U14-+): track 3.09 -> 0.00 mm
- net Net-(U11-+): track 3.09 -> 0.00 mm
- net Net-(R38-Pad1): track 2.33 -> 0.00 mm
- net Net-(R34-Pad1): track 2.33 -> 0.00 mm
- net SD_LP_FROM_HVD: track 13.5 -> 11.9 mm
- net Net-(D12-K): track 0.00 -> 1.46 mm
- net Upstream: track 19.2 -> 17.8 mm, vias 1 -> 0
- net SD_LP_IN: track 89.9 -> 88.6 mm
- net Local: track 23.8 -> 24.0 mm, vias 1 -> 0
- net GND: vias 48 -> 42
Other:
- outline, holes or cut-outs redrawn
- board text added: "BSPD"
