File: VehicleJunctionBoxMotherboard_PCB/VehicleJunctionBoxMotherboard_PCB.kicad_sch (KiCad schematic)
At the start: 41 parts, among them J1 HVD IL, J2 Vehicle, J3 TSMP+, J4 TSMP-, J5 HV+, J6 HV-, J7 TSMP GLV-, J9 Conn_01x07, Q1 SSM3J328R LF, U1 AMS1117-5.0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

Commit message: Optimised
Parts:
- removed C29, C30: 100n, Capacitor_SMD:C_0603_1608Metric, symbol Device:C_Small
- removed R33 (x4): 10k, Resistor_SMD:R_0603_1608Metric, symbol Device:R_Small
- removed R33 (x2): 5.6k, Resistor_SMD:R_0603_1608Metric, symbol Device:R_Small
- removed U10 (x2): TLV7031DBV, Package_TO_SOT_SMD:SOT-23-5, symbol Comparator:TLV7031DBV
- added D3: 771-PLVA650A, Package_TO_SOT_SMD:SOT-23, symbol Device:D_Zener
- added D5: Green, LED_SMD:LED_0603_1608Metric, symbol Device:LED_Small
- R33: value 10k -> 18k
- R33: value 10k -> 4.7k
Connections:
- net +5V: now also D3.3 (K)
- net GLV+: now also D5.2 (A); no longer R33.2
- net GND: now also D3.1 (A)
- net Local: now also J9.3 (Pin_3), R33.1, R33.2; no longer J9.2 (Pin_2)
- net Upstream: now also J9.2 (Pin_2), R33.1, R33.2; no longer J9.3 (Pin_3)
- new net: D5.1 (K), R33.2
Other:
- note added: "14V down to 3.3V"
- note removed: "14V down to 5V"
- note removed: "5/2 V Threshold"
- note removed: "5V to 3.3V"
- note removed: "When SD Loop is high, Output is High"
- moved on the sheet: C1, C2, C8, R33, U1
